Commit message: feature: navsat_to_odom converter and imu roll and pitch switcher added. Hesai OT128 point time_stamp support added to activate deskew function. config params tuned

File: config/robot.urdf.xacro (robot description, xacro)
@@ -9,8 +9,8 @@
     <origin xyz="0 0 0" rpy="0 0 0" />
   </joint>
-  <link name="lidar_link"> </link>
+  <link name="rs_helios_top_base_link"> </link>
   <joint name="lidar_joint" type="fixed">
     <parent link="base_link" />
-    <child link="lidar_link" />
+    <child link="rs_helios_top_base_link" />
     <origin xyz="0 0 0" rpy="0 0 0" />
   </joint>

Commit message: init first broken map

File: config/robot.urdf.xacro (robot description, xacro)
@@ -9,8 +9,14 @@
     <origin xyz="0 0 0" rpy="0 0 0" />
   </joint>
-  <link name="rs_helios_top_base_link"> </link>
+  <!-- <link name="rs_helios_top_base_link"> </link>
   <joint name="lidar_joint" type="fixed">
     <parent link="base_link" />
     <child link="rs_helios_top_base_link" />
+    <origin xyz="0 0 0" rpy="0 0 0" />
+  </joint> -->
+  <link name="hesai_ot128_top"> </link>
+  <joint name="lidar_joint" type="fixed">
+    <parent link="base_link" />
+    <child link="hesai_ot128_top" />
     <origin xyz="0 0 0" rpy="0 0 0" />
   </joint>

Commit message: push final map configs

File: config/robot.urdf.xacro (robot description, xacro)
@@ -19,5 +19,5 @@
     <parent link="base_link" />
     <child link="hesai_ot128_top" />
-    <origin xyz="0 0 0" rpy="0 0 0" />
+    <origin xyz="0 0 0" rpy="0 0 1.57079632679" />
   </joint>
   <link name="imu_link"> </link>

Commit message: sync with latest version

File: config/robot.urdf.xacro (robot description, xacro)
@@ -15,19 +15,19 @@
     <origin xyz="0 0 0" rpy="0 0 0" />
   </joint> -->
-  <link name="hesai_ot128_top"> </link>
+  <link name="rs_helios_top_base_link"> </link>
   <joint name="lidar_joint" type="fixed">
     <parent link="base_link" />
-    <child link="hesai_ot128_top" />
-    <origin xyz="0 0 0" rpy="0 0 1.57079632679" />
+    <child link="rs_helios_top_base_link" />
+    <origin xyz="0 0 0" rpy="0 0 0.0" />
   </joint>
-  <link name="imu_link"> </link>
+  <link name="imu_deneme_link"> </link>
   <joint name="imu_joint" type="fixed">
     <parent link="chassis_link" />
-    <child link="imu_link" />
+    <child link="imu_deneme_link" />
     <origin xyz="0 0 0" rpy="0 0 0" />
   </joint>
   <link name="laser_sensor_frame"> </link>
   <joint name="laser_joint" type="fixed">
-    <parent link="imu_link" />
+    <parent link="imu_deneme_link" />
     <child link="laser_sensor_frame" />
     <origin xyz="0 0 0" rpy="0 0 0" />

Commit message: fix: Update parameters in params.yaml and robot.urdf.xacro for lidar frame consistency; enhance map saving logic in mapOptimization.cpp

File: config/robot.urdf.xacro (robot description, xacro)
@@ -9,8 +9,8 @@
     <origin xyz="0 0 0" rpy="0 0 0" />
   </joint>
-  <link name="rs_helios_top_base_link"> </link>
+  <link name="hesai_ot128_top_base_link"> </link>
   <joint name="lidar_joint" type="fixed">
     <parent link="base_link" />
-    <child link="rs_helios_top_base_link" />
+    <child link="hesai_ot128_top_base_link" />
     <origin xyz="0 0 0" rpy="0 0 0" />
   </joint>

Commit message: fix: Update pointCloudTopic in params.yaml for consistency; modify robot.urdf.xacro for joint definitions and enhance rviz2.rviz with tracked objects visualization

File: config/robot.urdf.xacro (robot description, xacro)
@@ -1,35 +1,10 @@
 <?xml version="1.0"?>
 <robot name="lio" xmlns:xacro="http://tixiaoshan.github.io/">
-  <xacro:property name="PI" value="3.1415926535897931" />
-  <link name="chassis_link"></link>
-  <link name="base_link"></link>
-  <joint name="base_link_joint" type="fixed">
+  <link name="base_link"/>
+  <link name="hesai_ot128_top_base_link"/>
+  <joint name="lidar_joint" type="fixed">
     <parent link="base_link"/>
-    <child link="chassis_link" />
-    <origin xyz="0 0 0" rpy="0 0 0" />
-  </joint>
-  <link name="hesai_ot128_top_base_link"> </link>
-  <joint name="lidar_joint" type="fixed">
-    <parent link="base_link" />
-    <child link="hesai_ot128_top_base_link" />
-    <origin xyz="0 0 0" rpy="0 0 0" />
-  </joint>
-  <link name="imu_link"> </link>
-  <joint name="imu_joint" type="fixed">
-    <parent link="chassis_link" />
-    <child link="imu_link" />
-    <origin xyz="0 0 0" rpy="0 0 0" />
-  </joint>
-  <link name="laser_sensor_frame"> </link>
-  <joint name="laser_joint" type="fixed">
-    <parent link="imu_link" />
-    <child link="laser_sensor_frame" />
-    <origin xyz="0 0 0" rpy="0 0 0" />
-  </joint>
-  <link name="navsat_link"> </link>
-  <joint name="navsat_joint" type="fixed">
-    <parent link="chassis_link" />
-    <child link="navsat_link" />
-    <origin xyz="0 0 0" rpy="0 0 0" />
+    <child link="hesai_ot128_top_base_link"/>
+    <origin xyz="1.495 0.0 1.806530" rpy="-0.009587 0.017595 0.0"/>
   </joint>
 </robot>
